File: Dokumentation/schaltplan/schaltplan.kicad_sch (KiCad schematic)
At the start: 13 parts, among them J1 Raspberry_Pi_5, K1 Relais, M1 Servo 1, M2 Servo 2, M3 Servo 3, M4 Servo 4, M5 Motor_DC, U1 Logic Level Converter, U2 PCA9685 as Servo Driver

Commit message: Writing more doku
Parts:
- added K2: Pumpe-Relais, Relay_THT:Relay_SPDT_Finder_40.41, symbol Relay:FINDER-40.41
- added M6: Pumpe, symbol Motor:Motor_DC
- A1: value Arduino_Nano_Every -> Arduino Nano
- BT1: value 6V Battery -> 6V Batterie
- J1: value Raspberry_Pi_5 -> RaspberryPi 5
- K1: value Relais -> Hauptmotor-Relais
- M5: value Motor_DC -> Hauptmotor
- U2: value PCA9685 as Servo Driver -> PCA9685 als Servo Driver
Connections:
- net at A1.29 (GND), A1.4 (GND), J1.14 (GND)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: now also K2.A2
- net at A1.6 (D3): now also K2.A1
- net at BT1.1 (+), K1.11, M1.2 (+)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: now also K2.11
- net at BT1.2 (-), M1.3 (-), M2.3 (-)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: now also M6.2 (-)
- new net: K2.14, M6.1 (+)
